File: Kicad/main_kicad/near365.kicad_pcb (KiCad board)
At the start: 2 copper layers, 110.1 x 130.8 mm, 34 parts, among them J1 BMS power input, J2 USB_C_Receptacle_USB2.0_16P, SW1 Switch, SW2 Switch, SW3 SW_en, SW4 SW_boot, SW5 RotaryEncoder_Switch_MP, U1 ESP32-S3-WROOM-1, U2 TC00500, U3 CR2013-MI2120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

Commit message: Updated power, made changes to 3d front plate, added pull down r to encoder
Parts:
- added R7: 10kΩ, Resistor_THT:R_Axial_DIN0207_L6.3mm_D2.5mm_P7.62mm_Horizontal, B.Cu at (247.7, 166.7)
- added R8: 10kΩ, Resistor_THT:R_Axial_DIN0207_L6.3mm_D2.5mm_P7.62mm_Horizontal, B.Cu at (227.6, 150.0)
- added R9: 10kΩ, Resistor_THT:R_Axial_DIN0207_L6.3mm_D2.5mm_P7.62mm_Horizontal, B.Cu at (243.4, 152.4)
Routing:
- net RT_B: track 81.6 -> 132.0 mm
- net +3.3V: track 502.5 -> 551.1 mm, vias 10 -> 11
- net RT_SW: track 65.6 -> 93.6 mm, vias 1 -> 3
- net RT_A: track 115.8 -> 121.7 mm
- net TFT_BL: track 115.1 -> 119.5 mm, vias 6 -> 8
Other:
- outline, holes or cut-outs redrawn
